File: dab_mainboard.brd (EAGLE design)
At the start: 100 x 80 mm, 43 parts, among them J2 AVR_SPI_PROG_3X2PTH, U1 ATMEGA328P, U2 LSM9DS1, U3 PCA9306DCTR, Y1 16MHz

Commit message: Version 1 Final
Parts:
- removed J2: AVR_SPI_PROG_3X2PTH, SparkFun-Connectors:2X3
- added C15: 100n, resistor:C0603
- added C16, C17: 0.1u, resistor:C0603
- added ICSP: (no value), pinhead:2X03
- added R10, R11: 10k, rcl:R0603
- added S1, S2, S3: STANDOFF_ELECTRICAL, SparkFun-Electromechanical:STANDOFF-ELECTRICAL
- C5, C7: device resistor:C0603 -> resistor:C0805
- moved IO 111.9 mm to (40.0, 53.7)
- moved R9 104.8 mm to (52.6, 45.6), turned to 90 degrees
- moved SDA5 103.5 mm to (29.2, 34.0)
- moved SCL5 103.0 mm to (33.4, 35.3)
- moved SDA3 91.4 mm to (28.7, 27.9)
- moved SCL3 89.4 mm to (28.7, 29.1)
- moved +5V 87.4 mm to (34.6, 11.3), turned to 90 degrees
- moved +3.3V 83.9 mm to (9.14, 11.4), turned to 90 degrees
- moved SERIAL 74.9 mm to (4.06, 69.1), turned to 90 degrees
- moved KEYPAD 69.3 mm to (4.06, 42.3), turned to 90 degrees
- moved C2 64.7 mm to (8.38, 62.7), turned to 180 degrees
- moved C14 64.0 mm to (34.0, 22.7), turned to 180 degrees
- moved C13 61.0 mm to (34.0, 24.3), turned to 180 degrees
- moved PWR_IN 59.4 mm to (27.9, 2.54)
- moved C12 59.2 mm to (34.0, 27.3), turned to 180 degrees
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Connections:
- removed net CS_A/G: R7.1, U2.7
- new net N$4: R7.1, U2.6
- new net N$6: R11.1, U2.7
- new net N$7: R10.1, U2.5
- net +3V3: now also R10.2, R11.2
- net +5V: now also C15.1, C16.1, C17.1, ICSP.2; no longer J2.2
- net GND: now also C15.2, C16.2, C17.2, ICSP.6, S1.P1, S2.P1, S3.P1; no longer J2.6
- net MISO: now also ICSP.1; no longer J2.1
- net MOSI: now also ICSP.4; no longer J2.4
- net RST: now also ICSP.5; no longer J2.5
- net SCK: now also ICSP.3; no longer J2.3
Routing:
- net +5V: track 0.00 -> 240.3 mm, vias 0 -> 4
- net +3V3: track 0.00 -> 87.8 mm, vias 0 -> 5
- net RST: track 0.00 -> 57.5 mm, vias 0 -> 3
- net LED: track 0.00 -> 51.8 mm, vias 0 -> 2
- net N$11: track 0.00 -> 43.4 mm, vias 0 -> 2
- net VIN: track 0.00 -> 40.3 mm, vias 0 -> 2
- net LCD_RS: track 0.00 -> 36.1 mm, vias 0 -> 2
- net LCD_EN: track 0.00 -> 35.6 mm, vias 0 -> 2
- net LCD_DB7: track 0.00 -> 34.4 mm
- net SDA5V: track 0.00 -> 34.2 mm, vias 0 -> 2
- net LCD_DB6: track 0.00 -> 32.0 mm
- net SCL5V: track 0.00 -> 31.1 mm, vias 0 -> 2
- net RXI: track 0.00 -> 30.0 mm
- net LCD_DB5: track 0.00 -> 29.4 mm
- net LCD_DB4: track 0.00 -> 28.7 mm
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- added copper zone on layer 1, net GND
- added copper zone on layer 1, net N$12
- added copper zone on layer 1, net N$13
Other:
- board size 100 x 80 mm -> 60 x 80 mm
- board text added: "SAMTOMINDUSTRYS"
