File: dab_mainboard.sch (EAGLE design)
At the start: 43 parts, among them J2 AVR_SPI_PROG_3X2PTH, U1 ATMEGA328P, U2 LSM9DS1, U3 PCA9306DCTR, Y1 16MHz

Commit message: Version 1 Final
Parts:
- removed J2: AVR_SPI_PROG_3X2PTH, SparkFun-Connectors:AVR_SPI_PROG_3X2PTH
- added C15: 100n, resistor:C-EUC0603
- added C16, C17: 0.1u, resistor:C-EUC0603
- added ICSP: (no value), pinhead:PINHD-2X3
- added R10, R11: 10k, rcl:R-EU_R0603
- added S1, S2, S3: STANDOFF_ELECTRICAL, SparkFun-Electromechanical:STANDOFF_ELECTRICAL
- C5, C7: device resistor:C-EUC0603 -> resistor:C-EUC0805
Connections:
- removed net CS_A/G: R7.1, U2.CS_A/G
- new net N$4: R7.1, U2.SDO_M
- new net N$6: R11.1, U2.CS_A/G
- new net N$7: R10.1, U2.SDO_A/G
- net +3V3: now also R10.2, R11.2
- net +5V: now also C15.1, C16.1, C17.1, ICSP.2; no longer J2.2
- net GND: now also C15.2, C16.2, C17.2, ICSP.6, S1.P$1, S2.P$1, S3.P$1; no longer J2.6
- net MISO: now also ICSP.1; no longer J2.1
- net MOSI: now also ICSP.4; no longer J2.4
- net RST: now also ICSP.5; no longer J2.5
- net SCK: now also ICSP.3; no longer J2.3
Other:
- moved on the sheet: R7, R8
